Commit message: check

File: src/combat_robot_description/urdf/sensors.xacro (robot description, xacro)
@@ -30,5 +30,5 @@
     <parent link="base_link"/>
     <child link="imu_link"/>
-    <origin xyz="0 0 0.2" rpy="0 0 0"/> </joint>
+    <origin xyz="0.1 0 0.2" rpy="0 0 0"/> </joint>
   <gazebo reference="imu_link">
     <sensor name="imu_sensor" type="imu">
