Commit message: localization: gyro bias 보정 + GNSS heading 게이팅으로 yaw 안정화
- gyro_bias_comp.py (신규): xsens gyro z-bias 온라인 추정(정지 시 /odom 기준)
  → /imu/data_corrected 발행. 자력계 차폐로 gyro rate만 사용. 측정 bias 15.33°/min.
- ekf.yaml: ekf_odom/ekf_map가 보정 gyro(/imu/data_corrected, vyaw)로 회전 추적,
  GPS heading으로 절대 yaw, /imu/data orientation 미사용. 정지 drift 제거, 회전 map→odom<2°.
- gnss_heading.py: 속도 게이팅(이동 시만 heading 발행, 정지 시 차단해 q5 FLOAT drift 회피),
  circular-MA 평활, /odom·각속도 기반 게이팅, antenna offset 254.1→274 (q4 주행 보정).
- can_reader.py: 속도 threshold 기반 견고한 ZUPT 정지 판정.
- sensor.launch.py: gyro_bias_comp + 튜닝된 gnss_heading 파라미터 통합.
- 결과: 정지 안정, 직진 GPS 절대 yaw+위치, 회전 정확 추적.

Co-Authored-By: Claude Opus 4.8 (1M context) <noreply@anthropic.com>

File: src/combat_robot_description/urdf/sensors.xacro (robot description, xacro)
@@ -61,5 +61,5 @@
     <parent link="base_link"/>
     <child link="front_lidar_link"/>
-    <origin xyz="0.6 0 0.3" rpy="0 0 0"/> </joint>
+    <origin xyz="0.6 0 -0.1" rpy="0 0 0"/> </joint>
   <gazebo reference="front_lidar_link">
     <sensor name="front_lidar_sensor" type="gpu_lidar">
